File: tas5753.brd (EAGLE design)
At the start: 60.9 x 54.5 mm, 64 parts, among them IC1 AO4409, J6 JUMPER, P1 CONN_1X11_SMT_254, Q1 BSS138, U1 MAX16904RAUE33/V+, U2 TAS5753

Commit message: Add files via upload
Parts:
- C13, C29: value (none) -> 330u 35V
- moved C7 2.28 mm to (13.8, 13.0), turned to 270 degrees
- moved R6 2.19 mm to (14.7, 10.9), turned to 180 degrees
Connections:
- net N$2: now also C7.2, R6.2; no longer C7.1, R6.1
- net N$23: now also R6.1; no longer C7.2
- net N$4: now also C7.1; no longer R6.2
Routing:
- net N$7: track 0.77 -> 2.02 mm
- net 3.3V: track 78.6 -> 79.6 mm, vias 9 -> 10
- net GND: vias 86 -> 87
