File: tas5753.sch (EAGLE design)
At the start: 64 parts, among them IC1 AO4409, J6 JUMPER, P1 CONN_1X11_SMT_254, Q1 BSS138, U1 MAX16904RAUE33/V+, U2 TAS5753

Commit message: Add files via upload
Parts:
- C13, C29: value (none) -> 330u 35V
Connections:
- net N$2: now also C7.P$2, R6.2; no longer C7.P$1, R6.1
- net N$23: now also R6.1; no longer C7.P$2
- net N$4: now also C7.P$1; no longer R6.2
Other:
- moved on the sheet: C7, R6
Changed lines of the file:
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@@
 <part name="C5" library="hari" deviceset="CAP_CERAMIC" device="0603" value="4n7"/>
 <part name="C8" library="hari" deviceset="CAP_CERAMIC" device="0603" value="4n7"/>
-<part name="C13" library="SparkFun-Passives" deviceset="CAP_POL" device="E"/>
-<part name="C29" library="SparkFun-Passives" deviceset="CAP_POL" device="E"/>
+<part name="C13" library="SparkFun-Passives" deviceset="CAP_POL" device="E" value="330u 35V"/>
+<part name="C29" library="SparkFun-Passives" deviceset="CAP_POL" device="E" value="330u 35V"/>
 <part name="P1" library="hari" deviceset="CONN_1X11_SMT_254" device=""/>
 <part name="J2" library="Connector " deviceset="SCREW-TERMINAL-2P" device="'5.08'"/>
@@
 </plain>
 <instances>
-<instance part="R6" gate="G$1" x="40.64" y="25.4"/>
+<instance part="R6" gate="G$1" x="30.48" y="25.4"/>
 <instance part="R5" gate="G$1" x="12.7" y="17.78" rot="R90"/>
 <instance part="R9" gate="G$1" x="58.42" y="5.08" rot="R90"/>
@@
 </instance>
 <instance part="C31" gate="G$1" x="160.02" y="33.02" smashed="yes" rot="R180">
-<attribute name="NAME" x="167.64" y="33.02" size="1.27" layer="95" font="vector" rot="R180"/>
-<attribute name="VALUE" x="172.72" y="30.48" size="1.27" layer="96" font="vector" rot="R180"/>
+<attribute name="NAME" x="165.1" y="35.56" size="1.27" layer="95" font="vector" rot="R180"/>
+<attribute name="VALUE" x="172.72" y="33.02" size="1.27" layer="96" font="vector" rot="R180"/>
 </instance>
 <instance part="C4" gate="G$1" x="12.7" y="27.94" smashed="yes" rot="R180">
@@
 <attribute name="VALUE" x="10.16" y="27.94" size="1.27" layer="96" font="vector" rot="R180"/>
 </instance>
-<instance part="C7" gate="G$1" x="27.94" y="25.4" smashed="yes" rot="R270">
-<attribute name="NAME" x="30.48" y="27.94" size="1.27" layer="95" font="vector"/>
-<attribute name="VALUE" x="30.48" y="25.4" size="1.27" layer="96" font="vector"/>
+<instance part="C7" gate="G$1" x="40.64" y="22.86" smashed="yes" rot="R270">
+<attribute name="NAME" x="43.18" y="25.4" size="1.27" layer="95" font="vector"/>
+<attribute name="VALUE" x="38.1" y="25.4" size="1.27" layer="96" font="vector"/>
 </instance>
 <instance part="C5" gate="G$1" x="17.78" y="22.86" smashed="yes" rot="R180">
@@
 <instance part="C29" gate="G$1" x="154.94" y="33.02" smashed="yes">
 <attribute name="NAME" x="150.876" y="28.575" size="1.778" layer="95"/>
-<attribute name="VALUE" x="155.956" y="28.829" size="1.778" layer="96"/>
+<attribute name="VALUE" x="150.876" y="26.289" size="1.778" layer="96"/>
 </instance>
 <instance part="P1" gate="G$1" x="180.34" y="33.02" smashed="yes" rot="MR0"/>
@@
 </segment>
 </net>
-<net name="N$2" class="0">
-<segment>
-<pinref part="R6" gate="G$1" pin="1"/>
-<wire x1="33.02" y1="25.4" x2="35.56" y2="25.4" width="0.1524" layer="91"/>
-<pinref part="C7" gate="G$1" pin="P$1"/>
-</segment>
-</net>
 <net name="N$4" class="0">
 <segment>
-<pinref part="R6" gate="G$1" pin="2"/>
 <wire x1="38.1" y1="20.32" x2="45.72" y2="20.32" width="0.1524" layer="91"/>
 <wire x1="45.72" y1="20.32" x2="45.72" y2="22.86" width="0.1524" layer="91"/>
-<wire x1="45.72" y1="22.86" x2="45.72" y2="25.4" width="0.1524" layer="91"/>
 <wire x1="45.72" y1="22.86" x2="73.66" y2="22.86" width="0.1524" layer="91"/>
-<junction x="45.72" y="22.86"/>
 <pinref part="U2" gate="G$1" pin="PLLFLTP@PIN17"/>
 <pinref part="C8" gate="G$1" pin="P$1"/>
+<pinref part="C7" gate="G$1" pin="P$1"/>
+<junction x="45.72" y="22.86"/>
 </segment>
 </net>
@@
 <segment>
 <wire x1="30.48" y1="20.32" x2="25.4" y2="20.32" width="0.1524" layer="91"/>
-<wire x1="25.4" y1="20.32" x2="25.4" y2="25.4" width="0.1524" layer="91"/>
-<junction x="25.4" y="20.32"/>
 <wire x1="25.4" y1="15.24" x2="25.4" y2="20.32" width="0.1524" layer="91"/>
 <wire x1="25.4" y1="15.24" x2="48.26" y2="15.24" width="0.1524" layer="91"/>
@@
 <wire x1="48.26" y1="20.32" x2="73.66" y2="20.32" width="0.1524" layer="91"/>
 <pinref part="U2" gate="G$1" pin="ANAREG1@PIN18"/>
-<pinref part="C7" gate="G$1" pin="P$2"/>
 <pinref part="C8" gate="G$1" pin="P$2"/>
+<pinref part="R6" gate="G$1" pin="1"/>
+<wire x1="25.4" y1="25.4" x2="25.4" y2="20.32" width="0.1524" layer="91"/>
+<junction x="25.4" y="20.32"/>
 </segment>
 </net>
@@
 </segment>
 </net>
+<net name="N$2" class="0">
+<segment>
+<pinref part="R6" gate="G$1" pin="2"/>
+<pinref part="C7" gate="G$1" pin="P$2"/>
+<wire x1="35.56" y1="25.4" x2="38.1" y2="22.86" width="0.1524" layer="91"/>
+</segment>
+</net>
 </nets>
 </sheet>
 </sheets>
+<errors>
+</errors>
 </schematic>
 </drawing>
